File: pedalboard/Hauptwerk_Project_v2/Hauptwerk_Project.kicad_pcb (KiCad board)
At the start: 2 copper layers, 233.7 x 49.5 mm, 50 parts, among them J1 Power 5V, J2 1-6, J3 7-12, J4 13-18, J5 19-24, J6 25-30, J7 31-32, U1 74HC165, U2 74HC165, U3 74HC165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

Commit message: Fix vari
Parts:
- F1: value Fuse 2A / DC -> Fuse
- U5: value Arduino ProMicro -> ProMicro
Connections:
- U1 pad 7: Net-(U1-~{Q7}) -> unconnected-(U1-~{Q7}-Pad7)
- U1 pad 9: unconnected-(U1-Q7-Pad9) -> Net-(U1-Q7)
- U2 pad 10: Net-(U1-~{Q7}) -> Net-(U1-Q7)
- U2 pad 7: Net-(U2-~{Q7}) -> unconnected-(U2-~{Q7}-Pad7)
- U2 pad 9: unconnected-(U2-Q7-Pad9) -> Net-(U2-Q7)
- U3 pad 10: Net-(U2-~{Q7}) -> Net-(U2-Q7)
- U3 pad 7: Net-(U3-~{Q7}) -> unconnected-(U3-~{Q7}-Pad7)
- U3 pad 9: unconnected-(U3-Q7-Pad9) -> Net-(U3-Q7)
- U4 pad 10: Net-(U3-~{Q7}) -> Net-(U3-Q7)
Routing:
- net GND: track 0.00 -> 88.5 mm, vias 0 -> 4
- net Net-(U1-~{Q7}): track 44.0 -> 0.00 mm
- net Net-(U1-Q7): track 0.00 -> 42.6 mm
- net Net-(U3-~{Q7}): track 40.9 -> 0.00 mm
- net Net-(U2-~{Q7}): track 40.7 -> 0.00 mm
- net Net-(U2-Q7): track 0.00 -> 32.3 mm
- net Net-(U3-Q7): track 0.00 -> 32.1 mm
