File: pedalboard/Hauptwerk_Project_v2/Hauptwerk_Project.kicad_pcb (KiCad board)
At the start: 2 copper layers, 233.7 x 49.5 mm, 50 parts, among them J1 Power 5V, J2 1-6, J3 7-12, J4 13-18, J5 19-24, J6 25-30, J7 31-32, U1 74HC165, U2 74HC165, U3 74HC165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

Commit message: Update dim footprint
Parts:
- J1, J7: footprint TerminalBlock_Phoenix:TerminalBlock_Phoenix_MKDS-1,5-2-5.08_1x02_P5.08mm_Horizontal -> TerminalBlock_Phoenix:TerminalBlock_Phoenix_MPT-0,5-2-2.54_1x02_P2.54mm_Horizontal
- J2, J3, J4, J5, J6: footprint TerminalBlock_Phoenix:TerminalBlock_Phoenix_MKDS-1,5-6-5.08_1x06_P5.08mm_Horizontal -> TerminalBlock_Phoenix:TerminalBlock_Phoenix_MPT-0,5-6-2.54_1x06_P2.54mm_Horizontal
- moved J3 6.86 mm to (85.6, 99.1)
- moved J2 6.36 mm to (53.3, 99.3)
- moved J5 6.10 mm to (148.3, 99.1)
- moved J4 5.84 mm to (116.3, 99.1)
- moved J6 5.33 mm to (179.3, 99.1)
- moved J7 1.29 mm to (207.0, 99.1)
Routing:
- net Net-(J6-Pin_6): track 30.6 -> 33.6 mm
- net Net-(J2-Pin_6): track 50.4 -> 53.3 mm
- net Net-(J2-Pin_1): track 100.9 -> 103.7 mm
- net Net-(J3-Pin_1): track 46.6 -> 49.5 mm
- net Net-(J4-Pin_6): track 76.5 -> 79.3 mm
- net Net-(J5-Pin_6): track 29.4 -> 32.1 mm
- net Net-(J5-Pin_1): track 73.0 -> 75.5 mm
- net Net-(J4-Pin_1): track 42.8 -> 45.2 mm
- net Net-(J3-Pin_6): track 68.2 -> 70.6 mm
- net Net-(J6-Pin_1): track 78.0 -> 80.2 mm
- net Net-(J6-Pin_5): track 29.9 -> 31.9 mm
- net Net-(J2-Pin_2): track 95.7 -> 97.6 mm
- net Net-(J2-Pin_5): track 51.3 -> 53.2 mm
- net Net-(J3-Pin_2): track 43.7 -> 45.5 mm
- net Net-(J4-Pin_5): track 84.8 -> 86.6 mm
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
Commit message: problem fix
Changed lines of the file:
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@@
-	)
-	(segment
-		(start 210.82 99.2275)
-		(end 210.815 99.2325)
-		(width 0.2)
-		(layer "F.Cu")
-		(net 33)
 	)
 	(segment
@@
 		(width 0.2)
 		(layer "F.Cu")
-		(net 34)
-	)
-	(segment
-		(start 205.74 99.2275)
-		(end 205.735 99.2325)
-		(width 0.2)
-		(layer "F.Cu")
