File: pedalboard/Hauptwerk_Project_v2/Hauptwerk_Project.kicad_sch (KiCad schematic)
At the start: 45 parts, among them J1 Power 5V, J2 1-6, J3 7-12, J4 13-18, J5 19-24, J6 25-30, J7 31-32, U1 74HC165, U2 74HC165, U3 74HC165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

Commit message: Fix vari
Connections:
- net at U2.10 (DS): now also U1.9 (Q7); no longer U1.7 (~{Q7})
- net at U2.7 (~{Q7}): no longer U3.10 (DS)
- net at U2.9 (Q7): now also U3.10 (DS)
- net at U3.7 (~{Q7}): no longer U4.10 (DS)
- net at U3.9 (Q7): now also U4.10 (DS)
Changed lines of the file:
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@@
-	(wire
-		(pts
-			(xy 64.77 27.94) (xy 64.77 25.4)
-		)
-		(stroke
-			(width 0)
-			(type default)
-		)
-	)
 	(wire
 		(pts
@@
 	(wire
 		(pts
-			(xy 185.42 22.86) (xy 228.6 22.86)
-		)
-		(stroke
-			(width 0)
-			(type default)
-		)
-	)
-	(wire
-		(pts
 			(xy 193.04 106.68) (xy 193.04 95.25)
 		)
@@
 	(wire
 		(pts
+			(xy 62.23 25.4) (xy 62.23 27.94)
+		)
+		(stroke
+			(width 0)
+			(type default)
+		)
+	)
+	(wire
+		(pts
 			(xy 166.37 119.38) (xy 166.37 184.15)
 		)
@@
 	(wire
 		(pts
+			(xy 182.88 22.86) (xy 228.6 22.86)
+		)
+		(stroke
+			(width 0)
+			(type default)
+		)
+	)
+	(wire
+		(pts
 			(xy 185.42 66.04) (xy 162.56 66.04)
 		)
@@
 	(wire
 		(pts
+			(xy 62.23 25.4) (xy 111.76 25.4)
+		)
+		(stroke
+			(width 0)
+			(type default)
+		)
+	)
+	(wire
+		(pts
 			(xy 259.08 72.39) (xy 261.62 72.39)
 		)
@@
 	(wire
 		(pts
-			(xy 127 22.86) (xy 171.45 22.86)
-		)
-		(stroke
-			(width 0)
-			(type default)
-		)
-	)
-	(wire
-		(pts
 			(xy 25.4 27.94) (xy 30.48 27.94)
 		)
@@
 	(wire
 		(pts
-			(xy 64.77 25.4) (xy 111.76 25.4)
-		)
-		(stroke
-			(width 0)
-			(type default)
-		)
-	)
-	(wire
-		(pts
 			(xy 137.16 175.26) (xy 137.16 184.15)
 		)
@@
 	(wire
 		(pts
+			(xy 124.46 22.86) (xy 171.45 22.86)
+		)
+		(stroke
+			(width 0)
+			(type default)
+		)
+	)
+	(wire
+		(pts
 			(xy 200.66 106.68) (xy 200.66 99.06)
 		)
@@
 	(wire
 		(pts
+			(xy 124.46 22.86) (xy 124.46 27.94)
+		)
+		(stroke
+			(width 0)
+			(type default)
+		)
+	)
+	(wire
+		(pts
 			(xy 233.68 25.4) (xy 233.68 119.38)
 		)
@@
 	(wire
 		(pts
+			(xy 182.88 22.86) (xy 182.88 27.94)
+		)
+		(stroke
+			(width 0)
+			(type default)
+		)
+	)
+	(wire
+		(pts
 			(xy 243.84 53.34) (xy 243.84 69.85)
 		)
@@
 	(wire
 		(pts
-			(xy 185.42 27.94) (xy 185.42 22.86)
-		)
-		(stroke
-			(width 0)
-			(type default)
-		)
-	)
-	(wire
-		(pts
 			(xy 238.76 72.39) (xy 238.76 74.93)
 		)
@@
 		)
 		(stroke
-			(width 0)
-			(type default)
-		)
-	)
-	(wire
-		(pts
-			(xy 127 27.94) (xy 127 22.86)
-		)
-		(stroke
